File: catpad_PCB/catpad_PCB.kicad_sch (KiCad schematic)
At the start: 17 parts, among them SW1 SW_Push, SW2 SW_Push, SW3 SW_Push, SW4 SW_Push, SW5 SW_Push, SW6 SW_Push, SW7 SW_Push, SW8 SW_Push, U1 MOUDLE-SEEEDUINO-XIAO

Commit message: Finished the schem
Parts:
- added D10, D9: SK6812MINI-E, SK6812MINI-E - 3.2x2.8x1.78mm, symbol neopixel:SK6812MINI-E
Connections:
- net +5V: now also D10.1 (VDD), D9.1 (VDD)
- net GND: now also D10.3 (VSS), D9.3 (VSS)
- net NEO: now reaches U1.8 (PB09_A7_D7_RX)
- net NEO: now also D9.4 (DIN)
- new net: D10.4 (DIN), D9.2 (DOUT)
- no-connect marks 0 -> 1
Other:
- moved on the sheet: D1, D2, D3, D4, D5, D6, D7, D8, SW1, SW2, SW3, SW4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

Commit message: Finished the PCB
Parts:
- D1, D2, D3, D4, D5, D6, D7, D8: footprint (none) -> Diode_THT:D_DO-35_SOD27_P7.62mm_Horizontal
- D10, D9: footprint SK6812MINI-E - 3.2x2.8x1.78mm -> Care_package:SK6812MINI-E_fixed
- SW1, SW2, SW3, SW4, SW5, SW6, SW7, SW8: footprint (none) -> Button_Switch_Keyboard:SW_Cherry_MX_1.00u_PCB
- U1: footprint (none) -> Care_package:XIAO-Generic-Hybrid-14P-2.54-21X17.8MM
Other:
- added sheet MCU (MCU.kicad_sch)
- added sheet NEOs (NEOs.kicad_sch)
- added sheet Switchs (Switchs.kicad_sch)
- moved on the sheet: D10, D9

Commit message: Added 3D models to the PCB
Parts:
- SW1, SW2, SW3, SW4, SW5, SW6, SW7, SW8: footprint Button_Switch_Keyboard:SW_Cherry_MX_1.00u_PCB -> My_Footprints:SW_Cherry_MX_1.00u_PCB_With_3D
Changed lines of the file:
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@@
+	)
+	(junction
+		(at 116.84 67.31)
+		(diameter 0)
+		(color 0 0 0 0)
 	)
 	(junction
@@
 	)
 	(junction
-		(at 116.84 67.31)
-		(diameter 0)
-		(color 0 0 0 0)
-	)
-	(junction
 		(at 157.48 58.42)
 		(diameter 0)
@@
 	(wire
 		(pts
+			(xy 67.31 55.88) (xy 67.31 54.61)
+		)
+		(stroke
+			(width 0)
+			(type default)
+		)
+	)
+	(wire
+		(pts
+			(xy 147.32 67.31) (xy 163.83 67.31)
+		)
+		(stroke
+			(width 0)
+			(type default)
+		)
+	)
+	(wire
+		(pts
+			(xy 173.99 35.56) (xy 173.99 58.42)
+		)
+		(stroke
+			(width 0)
+			(type default)
+		)
+	)
+	(wire
+		(pts
+			(xy 142.24 35.56) (xy 142.24 58.42)
+		)
+		(stroke
+			(width 0)
+			(type default)
+		)
+	)
+	(wire
+		(pts
 			(xy 116.84 67.31) (xy 132.08 67.31)
-		)
-		(stroke
-			(width 0)
-			(type default)
-		)
-	)
-	(wire
-		(pts
-			(xy 67.31 55.88) (xy 67.31 54.61)
-		)
-		(stroke
-			(width 0)
-			(type default)
-		)
-	)
-	(wire
-		(pts
-			(xy 147.32 67.31) (xy 163.83 67.31)
-		)
-		(stroke
-			(width 0)
-			(type default)
-		)
-	)
-	(wire
-		(pts
-			(xy 173.99 35.56) (xy 173.99 58.42)
-		)
-		(stroke
-			(width 0)
-			(type default)
-		)
-	)
-	(wire
-		(pts
-			(xy 142.24 35.56) (xy 142.24 58.42)
 		)
 		(stroke
@@
 			)
 		)
-		(property "Footprint" "Button_Switch_Keyboard:SW_Cherry_MX_1.00u_PCB"
+		(property "Footprint" "My_Footprints:SW_Cherry_MX_1.00u_PCB_With_3D"
 			(at 137.16 53.34 0)
 			(effects
@@
 			)
 		)
-		(property "Footprint" "Button_Switch_Keyboard:SW_Cherry_MX_1.00u_PCB"
+		(property "Footprint" "My_Footprints:SW_Cherry_MX_1.00u_PCB_With_3D"
 			(at 137.16 30.48 0)
 			(effects
@@
 			)
 		)
-		(property "Footprint" "Button_Switch_Keyboard:SW_Cherry_MX_1.00u_PCB"
+		(property "Footprint" "My_Footprints:SW_Cherry_MX_1.00u_PCB_With_3D"
 			(at 168.91 30.48 0)
 			(effects
@@
 			)
 		)
-		(property "Footprint" "Button_Switch_Keyboard:SW_Cherry_MX_1.00u_PCB"
+		(property "Footprint" "My_Footprints:SW_Cherry_MX_1.00u_PCB_With_3D"
 			(at 168.91 53.34 0)
 			(effects
@@
 			)
 		)
-		(property "Footprint" "Button_Switch_Keyboard:SW_Cherry_MX_1.00u_PCB"
+		(property "Footprint" "My_Footprints:SW_Cherry_MX_1.00u_PCB_With_3D"
 			(at 152.4 30.48 0)
 			(effects
@@
 			)
 		)
-		(property "Footprint" "Button_Switch_Keyboard:SW_Cherry_MX_1.00u_PCB"
+		(property "Footprint" "My_Footprints:SW_Cherry_MX_1.00u_PCB_With_3D"
 			(at 121.92 30.48 0)
 			(effects
@@
 			)
 		)
-		(property "Footprint" "Button_Switch_Keyboard:SW_Cherry_MX_1.00u_PCB"
+		(property "Footprint" "My_Footprints:SW_Cherry_MX_1.00u_PCB_With_3D"
 			(at 152.4 53.34 0)
 			(effects
@@
 			)
 		)
-		(property "Footprint" "Button_Switch_Keyboard:SW_Cherry_MX_1.00u_PCB"
+		(property "Footprint" "My_Footprints:SW_Cherry_MX_1.00u_PCB_With_3D"
 			(at 121.92 53.34 0)
 			(effects
